File: PCB Design/Teensy Board/Teensy_board.sch (EAGLE design)
At the start: 32 parts, among them IC1 MC7805BDTRKG, IC2 UA78M33CKVU, U1 PCA9685PW, U2 74HC4051PW,118, U3 74HC4051PW,118, X1 RJ45-8X, X2 RJ45-8X, X3 RJ45-8X, X4 RJ45-8X, X5 RJ45-8X, X6 RJ45-8X

Commit message: teensy PCB
Parts:
- removed JP1: (no value), jumper:JP2E
- removed T1: (no value), CBLA_Test_bed_Library:NTD5867NLT4G
- added Q1: (no value), transistors:2N7002_SOT23
- added SV1: (no value), con-lstb:MA04-1
- added SV2: (no value), con-lstb:MA04-2
- added SV3, SV4, SV5, SV6, SV7, SV8: (no value), con-lstb:MA08-1
Connections:
- removed net A6: U$2.20/A6/PWM, X6.5
- removed net A7: U$2.21/A7/PWM, X6.6
- removed net FPWM_3_1: U$2.22/A8/T/PWM, X3.1
- removed net FPWM_3_2: U$2.23/A9/T/PWM, X3.2
- removed net N$1: U1.LED0, X1.3
- removed net N$11: U1.LED8, X5.1
- removed net N$12: U1.LED9, X5.2
- removed net N$13: U1.LED10, X5.3
- removed net N$14: U1.LED11, X5.4
- removed net N$15: U1.LED12, X6.1
- removed net N$16: U1.LED13, X6.2
- removed net N$17: U1.LED14, X6.3
- removed net N$2: U1.LED1, X1.4
- removed net N$20: R6.2, T1.G
- removed net N$3: U1.LED2, X2.3
- removed net N$33: U1.LED15
- removed net N$4: U1.LED3, X2.4
- removed net N$5: U1.LED4, X3.3
- removed net N$6: U1.LED5, X3.4
- removed net N$7: U1.LED6, X4.3
- removed net N$8: U1.LED7, X4.4
- removed net PWR_LED_GND: JP1.3, R1.1
- new net A8: SV6.5, U$2.22/A8/T/PWM, X4.5
- new net A9: SV6.6, U$2.23/A9/T/PWM, X4.6
- new net CE: SV2.3, U$2.9/RX2/PWM
- new net CSN: SV2.4, U$2.10/TX2/PWM
- new net FPWM_5_1: SV7.1, U$2.25/T/PWM, X5.1
- new net FPWM_5_2: SV7.2, U$2.32/T/PWM, X5.2
- new net MISO: SV2.7, U$2.12/MISO
- new net MOSI: SV2.6, U$2.11/MOSI
- new net PGM_DO: Q1.G, R6.2, U$2.0/RX1/T
- new net SCK: SV2.5, U$2.13/SCK/LED
- new net SPWM_1_1: SV3.3, U1.LED0, X1.3
- new net SPWM_1_2: SV3.4, U1.LED1, X1.4
- new net SPWM_2_1: SV4.3, U1.LED2, X2.3
- new net SPWM_2_2: SV4.4, U1.LED3, X2.4
- new net SPWM_3_1: SV5.1, U1.LED4, X3.1
- new net SPWM_3_2: SV5.2, U1.LED5, X3.2
- new net SPWM_3_3: SV5.3, U1.LED6, X3.3
- new net SPWM_3_4: SV5.4, U1.LED7, X3.4
- new net SPWM_4_1: SV6.3, U1.LED14, X4.3
- new net SPWM_4_2: SV6.4, U1.LED15, X4.4
- new net SPWM_5_1: SV7.3, U1.LED12, X5.3
- new net SPWM_5_2: SV7.4, U1.LED13, X5.4
- new net SPWM_6_1: SV8.1, U1.LED8, X6.1
- new net SPWM_6_2: SV8.2, U1.LED9, X6.2
- new net SPWM_6_3: SV8.3, U1.LED10, X6.3
- new net SPWM_6_4: SV8.4, U1.LED11, X6.4
- net 3V3INT: now also SV1.4, SV2.2
- net A0: now also SV8.5, X6.5; no longer X1.5
- net A1: now also SV8.6, X6.6; no longer X1.6
- net A12: now also SV4.5, X2.5; no longer X3.5
- net A13: now also SV3.5, X1.5; no longer X3.6
- net A15: now also SV4.6, X2.6; no longer X4.5
- net A16: now also SV5.5, X3.5; no longer X5.5
- net A17: now also SV5.6, X3.6; no longer X5.6
- net A2: now also SV7.5, X5.5; no longer X2.5
- net A20: now also SV3.6, X1.6; no longer X4.6
- net A3: now also SV7.6, X5.6; no longer X2.6
- net FPWM_1_1: now also SV3.1
- net FPWM_1_2: now also SV3.2
- net FPWM_2_1: now also SV4.1
- net FPWM_2_2: now also SV4.2
- net FPWM_4_1: now also SV6.1, U$2.20/A6/PWM; no longer U$2.25/T/PWM
- net FPWM_4_2: now also SV6.2, U$2.21/A7/PWM; no longer U$2.32/T/PWM
- net GND: now also Q1.S, R1.1, SV1.1, SV2.1; no longer JP1.2, T1.S
- net MUL_SCL_1: now also SV3.7, U3.Y4; no longer U3.Y0
- net MUL_SCL_2: now also SV4.7, U3.Y6; no longer U3.Y1
- net MUL_SCL_3: now also SV5.7, U3.Y7; no longer U3.Y2
- net MUL_SCL_4: now also SV6.7, U3.Y2; no longer U3.Y3
- net MUL_SCL_5: now also SV7.7, U3.Y1; no longer U3.Y4
- net MUL_SCL_6: now also SV8.7, U3.Y0; no longer U3.Y5
- net MUL_SDA_1: now also SV3.8, U2.Y4; no longer U2.Y0
- net MUL_SDA_2: now also SV4.8, U2.Y6; no longer U2.Y1
- net MUL_SDA_3: now also SV5.8, U2.Y7; no longer U2.Y2
- net MUL_SDA_4: now also SV6.8, U2.Y2; no longer U2.Y3
- net MUL_SDA_5: now also SV7.8, U2.Y1; no longer U2.Y4
- net MUL_SDA_6: now also SV8.8, U2.Y0; no longer U2.Y5
- net PGM: now also Q1.D; no longer T1.D
- net SCL_PWM: now also SV1.2
- net SDA_PWM: now also SV1.3
Other:
- moved on the sheet: C1, C2, C3, C4, C5, D1, IC1, IC2, LED1, LED2, LED3, R1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

Commit message: Teensy Board
Connections:
- removed net A20: SV3.6, U$2.31/A20, X1.6
- new net A11: SV3.5, U$2.A11, X1.5
- net +3V3: now also LED3.A; no longer LED2.A
- net +5V: now also LED2.A; no longer LED3.A
- net A13: now also SV3.6, X1.6; no longer SV3.5, X1.5
- net FPWM_2_1: now also U$2.6/PWM; no longer U$2.5/PWM
- net FPWM_2_2: now also U$2.5/PWM; no longer U$2.6/PWM
- net N$18: now also LED3.C; no longer LED2.C
- net N$19: now also LED2.C; no longer LED3.C
- net PGM_DO: now also U$2.7/RX3; no longer U$2.0/RX1/T
- net SCL_PWM: now also SV1.3; no longer SV1.2
- net SDA_PWM: now also SV1.2; no longer SV1.3
Other:
- moved on the sheet: LED2, LED3
Changed lines of the file:
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@@
 <part name="C4" library="rcl" deviceset="C-US" device="C0603" value="100nF"/>
 <part name="C5" library="rcl" deviceset="C-US" device="C0603" value="100nF"/>
+<part name="LED3" library="led" deviceset="LED" device="SML1206"/>
+<part name="R4" library="CBLA_Test_bed_Library" deviceset="R-US_" device="R0603" value="470"/>
 <part name="LED2" library="led" deviceset="LED" device="SML1206"/>
-<part name="R4" library="CBLA_Test_bed_Library" deviceset="R-US_" device="R0603" value="470"/>
-<part name="LED3" library="led" deviceset="LED" device="SML1206"/>
 <part name="R5" library="CBLA_Test_bed_Library" deviceset="R-US_" device="R0603" value="470"/>
 <part name="JP2" library="jumper" deviceset="JP2E" device=""/>
@@
 <instance part="C4" gate="G$1" x="195.58" y="24.13"/>
 <instance part="C5" gate="G$1" x="140.97" y="25.4"/>
-<instance part="LED2" gate="G$1" x="125.73" y="30.48"/>
+<instance part="LED3" gate="G$1" x="125.73" y="30.48"/>
 <instance part="R4" gate="G$1" x="125.73" y="19.05" rot="R90"/>
-<instance part="LED3" gate="G$1" x="180.34" y="30.48"/>
+<instance part="LED2" gate="G$1" x="180.34" y="30.48"/>
 <instance part="R5" gate="G$1" x="180.34" y="19.05" rot="R90"/>
 <instance part="JP2" gate="1" x="189.23" y="156.21" rot="R180"/>
@@
 <pinref part="IC1" gate="G$1" pin="VO"/>
 <wire x1="187.96" y1="33.02" x2="180.34" y2="33.02" width="0.1524" layer="91"/>
-<pinref part="LED3" gate="G$1" pin="A"/>
+<pinref part="LED2" gate="G$1" pin="A"/>
 <wire x1="180.34" y1="33.02" x2="175.26" y2="33.02" width="0.1524" layer="91"/>
 <junction x="180.34" y="33.02"/>
@@
 <wire x1="125.73" y1="33.02" x2="120.65" y2="33.02" width="0.1524" layer="91"/>
 <wire x1="140.97" y1="27.94" x2="140.97" y2="33.02" width="0.1524" layer="91"/>
-<pinref part="LED2" gate="G$1" pin="A"/>
+<pinref part="LED3" gate="G$1" pin="A"/>
 <junction x="125.73" y="33.02"/>
 <pinref part="C5" gate="G$1" pin="1"/>
@@
 </segment>
 <segment>
-<pinref part="SV1" gate="1" pin="3"/>
-<wire x1="191.77" y1="90.17" x2="194.31" y2="90.17" width="0.1524" layer="91"/>
-<label x="195.58" y="90.17" size="1.778" layer="95"/>
+<pinref part="SV1" gate="1" pin="2"/>
+<wire x1="191.77" y1="87.63" x2="194.31" y2="87.63" width="0.1524" layer="91"/>
+<label x="195.58" y="87.63" size="1.778" layer="95"/>
 </segment>
 </net>
@@
 </segment>
 <segment>
-<pinref part="SV1" gate="1" pin="2"/>
-<wire x1="191.77" y1="87.63" x2="194.31" y2="87.63" width="0.1524" layer="91"/>
-<label x="195.58" y="87.63" size="1.778" layer="95"/>
+<pinref part="SV1" gate="1" pin="3"/>
+<wire x1="191.77" y1="90.17" x2="194.31" y2="90.17" width="0.1524" layer="91"/>
+<label x="195.58" y="90.17" size="1.778" layer="95"/>
 </segment>
 </net>
@@
 </segment>
 <segment>
-<pinref part="U$2" gate="G$1" pin="5/PWM"/>
-<wire x1="107.95" y1="171.45" x2="101.6" y2="171.45" width="0.1524" layer="91"/>
-<label x="86.36" y="171.45" size="1.778" layer="95"/>
+<pinref part="U$2" gate="G$1" pin="6/PWM"/>
+<wire x1="107.95" y1="168.91" x2="101.6" y2="168.91" width="0.1524" layer="91"/>
+<label x="86.36" y="168.91" size="1.778" layer="95"/>
 </segment>
 </net>
@@
 </segment>
 <segment>
-<pinref part="U$2" gate="G$1" pin="6/PWM"/>
-<wire x1="107.95" y1="168.91" x2="101.6" y2="168.91" width="0.1524" layer="91"/>
-<label x="86.36" y="168.91" size="1.778" layer="95"/>
+<pinref part="U$2" gate="G$1" pin="5/PWM"/>
+<wire x1="107.95" y1="171.45" x2="101.6" y2="171.45" width="0.1524" layer="91"/>
+<label x="86.36" y="171.45" size="1.778" layer="95"/>
 </segment>
 </net>
@@
 </segment>
 <segment>
-<pinref part="X1" gate="G$1" pin="5"/>
-<wire x1="35.56" y1="179.07" x2="41.91" y2="179.07" width="0.1524" layer="91"/>
-<label x="43.18" y="179.07" size="1.778" layer="95"/>
-<pinref part="SV3" gate="1" pin="5"/>
-<wire x1="21.59" y1="179.07" x2="35.56" y2="179.07" width="0.1524" layer="91"/>
-<junction x="35.56" y="179.07"/>
+<pinref part="X1" gate="G$1" pin="6"/>
+<wire x1="35.56" y1="176.53" x2="41.91" y2="176.53" width="0.1524" layer="91"/>
+<label x="43.18" y="176.53" size="1.778" layer="95"/>
+<pinref part="SV3" gate="1" pin="6"/>
+<wire x1="21.59" y1="176.53" x2="35.56" y2="176.53" width="0.1524" layer="91"/>
+<junction x="35.56" y="176.53"/>
 </segment>
 </net>
@@
 </segment>
 </net>
-<net name="A20" class="0">
-<segment>
-<pinref part="U$2" gate="G$1" pin="31/A20"/>
-<wire x1="153.67" y1="138.43" x2="160.02" y2="138.43" width="0.1524" layer="91"/>
-<label x="161.29" y="138.43" size="1.778" layer="95"/>
-</segment>
-<segment>
-<pinref part="X1" gate="G$1" pin="6"/>
-<wire x1="35.56" y1="176.53" x2="41.91" y2="176.53" width="0.1524" layer="91"/>
-<label x="43.18" y="176.53" size="1.778" layer="95"/>
-<pinref part="SV3" gate="1" pin="6"/>
-<wire x1="21.59" y1="176.53" x2="35.56" y2="176.53" width="0.1524" layer="91"/>
-<junction x="35.56" y="176.53"/>
-</segment>
-</net>
 <net name="MUL_SCL_4" class="0">
 <segment>
@@
 <net name="N$18" class="0">
 <segment>
-<pinref part="LED2" gate="G$1" pin="C"/>
+<pinref part="LED3" gate="G$1" pin="C"/>
 <pinref part="R4" gate="G$1" pin="2"/>
 <pinref part="R4" gate="G$1" pin="2"/>
@@
 <net name="N$19" class="0">
 <segment>
-<pinref part="LED3" gate="G$1" pin="C"/>
+<pinref part="LED2" gate="G$1" pin="C"/>
 <pinref part="R5" gate="G$1" pin="2"/>
 <pinref part="R5" gate="G$1" pin="2"/>
@@
 <net name="PGM_DO" class="0">
 <segment>
-<pinref part="U$2" gate="G$1" pin="0/RX1/T"/>
-<wire x1="107.95" y1="184.15" x2="101.6" y2="184.15" width="0.1524" layer="91"/>
-<label x="86.36" y="184.15" size="1.778" layer="95"/>
-</segment>
-<segment>
 <wire x1="154.94" y1="80.01" x2="153.67" y2="80.01" width="0.1524" layer="91"/>
 <pinref part="R6" gate="G$1" pin="2"/>
@@
 <pinref part="Q1" gate="G$1" pin="G"/>
 </segment>
+<segment>
+<pinref part="U$2" gate="G$1" pin="7/RX3"/>
+<wire x1="107.95" y1="166.37" x2="101.6" y2="166.37" width="0.1524" layer="91"/>
+<label x="86.36" y="166.37" size="1.778" layer="95"/>
+</segment>
 </net>
 <net name="SCK" class="0">
@@
 </segment>
 </net>
+<net name="A11" class="0">
+<segment>
+<pinref part="U$2" gate="G$1" pin="A11"/>
+<wire x1="153.67" y1="151.13" x2="160.02" y2="151.13" width="0.1524" layer="91"/>
+<label x="161.29" y="151.13" size="1.778" layer="95"/>
+</segment>
+<segment>
+<pinref part="X1" gate="G$1" pin="5"/>
+<wire x1="35.56" y1="179.07" x2="41.91" y2="179.07" width="0.1524" layer="91"/>
+<label x="43.18" y="179.07" size="1.778" layer="95"/>
+<pinref part="SV3" gate="1" pin="5"/>
+<wire x1="21.59" y1="179.07" x2="35.56" y2="179.07" width="0.1524" layer="91"/>
+<junction x="35.56" y="179.07"/>
+</segment>
+</net>

Commit message: Teensy Board
Parts:
- added X8: UART, CBLA_Test_bed_Library:PINHD-1X2
- Q1: value (none) -> PROGRAM_FET
- SV1: value (none) -> PWM_I2C
- SV2: value (none) -> SPI
Connections:
- new net RX1: U$2.0/RX1/T, X8.2
- new net TX1: U$2.1/TX1/T, X8.1
Other:
- note added: "ISP"
- moved on the sheet: Q1, R6
Changed lines of the file:
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@@
 <setting verticaltext="up"/>
 </settings>
-<grid distance="0.05" unitdist="inch" unit="inch" style="lines" multiple="1" display="no" altdistance="0.025" altunitdist="inch" altunit="inch"/>
+<grid distance="0.1" unitdist="inch" unit="inch" style="lines" multiple="1" display="no" altdistance="0.01" altunitdist="inch" altunit="inch"/>
 <layers>
 <layer number="1" name="Top" color="4" fill="1" visible="no" active="no"/>
@@
 <part name="GND8" library="supply1" deviceset="GND" device=""/>
 <part name="R6" library="CBLA_Test_bed_Library" deviceset="R-US_" device="R0603" value="4k7"/>
-<part name="Q1" library="transistors" deviceset="2N700*" device="_SOT23" technology="2"/>
+<part name="Q1" library="transistors" deviceset="2N700*" device="_SOT23" technology="2" value="PROGRAM_FET"/>
 <part name="GND2" library="supply1" deviceset="GND" device=""/>
-<part name="SV1" library="con-lstb" deviceset="MA04-1" device=""/>
+<part name="SV1" library="con-lstb" deviceset="MA04-1" device="" value="PWM_I2C"/>
 <part name="GND9" library="supply1" deviceset="GND" device=""/>
-<part name="SV2" library="con-lstb" deviceset="MA04-2" device=""/>
+<part name="SV2" library="con-lstb" deviceset="MA04-2" device="" value="SPI"/>
 <part name="GND10" library="supply1" deviceset="GND" device=""/>
 <part name="SV3" library="con-lstb" deviceset="MA08-1" device=""/>
@@
 <part name="SV7" library="con-lstb" deviceset="MA08-1" device=""/>
 <part name="SV8" library="con-lstb" deviceset="MA08-1" device=""/>
+<part name="X8" library="CBLA_Test_bed_Library" deviceset="PINHD-1X2" device="" value="UART"/>
 </parts>
 <sheets>
@@
 <text x="208.28" y="10.16" size="2.54" layer="91">Mo Memarian
 2014-08-12</text>
+<text x="271.78" y="96.52" size="1.778" layer="91">ISP</text>
 </plain>
 <instances>
@@
 <instance part="GND7" gate="1" x="170.18" y="167.64"/>
 <instance part="P+5" gate="1" x="191.77" y="193.04"/>
-<instance part="GND8" gate="1" x="165.1" y="63.5"/>
-<instance part="R6" gate="G$1" x="158.75" y="69.85" rot="R180"/>
-<instance part="Q1" gate="G$1" x="165.1" y="82.55"/>
+<instance part="GND8" gate="1" x="157.48" y="60.96"/>
+<instance part="R6" gate="G$1" x="151.13" y="67.31" rot="R180"/>
+<instance part="Q1" gate="G$1" x="157.48" y="80.01" smashed="yes">
+<attribute name="NAME" x="164.084" y="80.772" size="1.778" layer="95"/>
+<attribute name="VALUE" x="161.544" y="73.406" size="1.778" layer="96"/>
+</instance>
 <instance part="GND2" gate="1" x="110.49" y="8.89"/>
-<instance part="SV1" gate="1" x="184.15" y="90.17"/>
+<instance part="SV1" gate="1" x="184.15" y="90.17" smashed="yes">
+<attribute name="VALUE" x="171.45" y="87.63" size="1.778" layer="96"/>
+<attribute name="NAME" x="182.88" y="96.012" size="1.778" layer="95"/>
+</instance>
 <instance part="GND9" gate="1" x="194.31" y="80.01"/>
 <instance part="SV2" gate="G$1" x="237.49" y="91.44"/>
@@
 <instance part="SV7" gate="1" x="13.97" y="69.85" rot="MR180"/>
 <instance part="SV8" gate="1" x="13.97" y="41.91" rot="MR180"/>
+<instance part="X8" gate="G$1" x="175.26" y="111.76" rot="R180"/>
 </instances>
 <busses>
@@
 <segment>
 <pinref part="GND8" gate="1" pin="GND"/>
-<wire x1="165.1" y1="72.39" x2="165.1" y2="69.85" width="0.1524" layer="91"/>
+<wire x1="157.48" y1="69.85" x2="157.48" y2="67.31" width="0.1524" layer="91"/>
 <pinref part="R6" gate="G$1" pin="1"/>
-<wire x1="165.1" y1="69.85" x2="165.1" y2="66.04" width="0.1524" layer="91"/>
-<wire x1="163.83" y1="69.85" x2="165.1" y2="69.85" width="0.1524" layer="91"/>
+<wire x1="157.48" y1="67.31" x2="157.48" y2="63.5" width="0.1524" layer="91"/>
+<wire x1="156.21" y1="67.31" x2="157.48" y2="67.31" width="0.1524" layer="91"/>
 <pinref part="Q1" gate="G$1" pin="S"/>
-<junction x="165.1" y="69.85"/>
+<junction x="157.48" y="67.31"/>
 </segment>
 <segment>
@@
 </segment>
 <segment>
-<label x="165.1" y="97.79" size="1.778" layer="95"/>
+<label x="157.48" y="95.25" size="1.778" layer="95"/>
 <pinref part="Q1" gate="G$1" pin="D"/>
-<wire x1="165.1" y1="92.71" x2="165.1" y2="96.52" width="0.1524" layer="91"/>
+<wire x1="157.48" y1="90.17" x2="157.48" y2="93.98" width="0.1524" layer="91"/>
 </segment>
 </net>
 <net name="PGM_DO" class="0">
 <segment>
-<wire x1="154.94" y1="80.01" x2="153.67" y2="80.01" width="0.1524" layer="91"/>
+<wire x1="147.32" y1="77.47" x2="146.05" y2="77.47" width="0.1524" layer="91"/>
 <pinref part="R6" gate="G$1" pin="2"/>
-<wire x1="153.67" y1="69.85" x2="153.67" y2="80.01" width="0.1524" layer="91"/>
-<wire x1="153.67" y1="80.01" x2="148.59" y2="80.01" width="0.1524" layer="91"/>
-<junction x="153.67" y="80.01"/>
-<label x="137.16" y="80.01" size="1.778" layer="95"/>
+<wire x1="146.05" y1="67.31" x2="146.05" y2="77.47" width="0.1524" layer="91"/>
+<wire x1="146.05" y1="77.47" x2="140.97" y2="77.47" width="0.1524" layer="91"/>
+<junction x="146.05" y="77.47"/>
+<label x="134.62" y="74.93" size="1.778" layer="95"/>
 <pinref part="Q1" gate="G$1" pin="G"/>
 </segment>
@@
 </segment>
 </net>
+<net name="RX1" class="0">
+<segment>
+<pinref part="U$2" gate="G$1" pin="0/RX1/T"/>
+<wire x1="107.95" y1="184.15" x2="101.6" y2="184.15" width="0.1524" layer="91"/>
+<label x="86.36" y="184.15" size="1.778" layer="95"/>
+</segment>
+<segment>
+<pinref part="X8" gate="G$1" pin="2"/>
+<wire x1="177.8" y1="111.76" x2="185.42" y2="111.76" width="0.1524" layer="91"/>
+<label x="187.96" y="111.76" size="1.778" layer="95"/>
+</segment>
+</net>
+<net name="TX1" class="0">
+<segment>
+<pinref part="U$2" gate="G$1" pin="1/TX1/T"/>
+<wire x1="107.95" y1="181.61" x2="101.6" y2="181.61" width="0.1524" layer="91"/>
+<label x="86.36" y="181.61" size="1.778" layer="95"/>
+</segment>
+<segment>
+<pinref part="X8" gate="G$1" pin="1"/>
+<wire x1="177.8" y1="109.22" x2="185.42" y2="109.22" width="0.1524" layer="91"/>
+<label x="187.96" y="109.22" size="1.778" layer="95"/>
+</segment>
+</net>
