File: Hardware/PCB Design/Tentacle Module/tentacle_module.brd (EAGLE design)
At the start: 101.6 x 30.5 mm, 56 parts, among them IC1 OKR-T/10-W12, IC2 MC7805BDTRKG, IC3 UA78M33CKVU, T1 NTD5867NL, T2 NTD5867NL, T3 NTD5867NL, T4 NTD5867NL, X3 RJ45-8X, X5 RJ45-8X

Commit message: Updated the board design
Parts:
- moved X5 8.64 mm to (27.1, 27.1)
Routing:
- net +12V: track 85.6 -> 67.1 mm
- net SDA: track 22.5 -> 32.6 mm, vias 0 -> 1
- net +5V: track 104.3 -> 113.0 mm
- net +3.3V: track 71.3 -> 79.6 mm
- net IR2: track 27.9 -> 34.2 mm
- net PWM3: track 36.0 -> 41.3 mm, vias 0 -> 1
- net +5V_HI-PWR: track 98.5 -> 103.4 mm
- net PWM1: track 37.1 -> 41.4 mm, vias 0 -> 1
- net PWM2: track 43.5 -> 47.1 mm
- net SCL: track 35.5 -> 38.6 mm
- net IR1: track 52.7 -> 55.1 mm
- net PWM4: track 32.0 -> 29.5 mm
- net PWR_LED_GND: track 22.1 -> 20.8 mm
- net GND: vias 26 -> 28
- added copper zone on layer 1, net +12V
- added copper zone on layer 16, net +12V
Other:
- board text added: "10/2014"
- board text added: "by PBAI & UWaterloo"
- board text removed: "08/2014"
