File: Hardware/PCB Design/Tentacle Tip/tentacle_tip.brd (EAGLE design)
At the start: 45.7 x 15.2 mm, 8 parts, among them U1 ADXL345

Commit message: Updated the board design
Parts:
- removed X1: (no value), CBLA_Test_bed_Library:MA04-2
- added X3: RJ45-8X, CBLA_Test_bed_Library:RJ45-NO-SHIELD
Connections:
- net +3.3V: now also X3.1; no longer X1.1
- net +5V: now also X3.3; no longer X1.3
- net GND: now also X3.2; no longer X1.2
- net IR2: now also X3.4; no longer X1.4
- net SCL: now also X3.5; no longer X1.5
- net SDA: now also X3.6; no longer X1.6
Routing:
- net SCL: track 24.1 -> 35.4 mm, vias 1 -> 2
- net IR2: track 27.0 -> 17.9 mm
- net +5V: track 9.53 -> 17.0 mm
- net +3.3V: track 45.4 -> 52.6 mm
- net GND: track 24.4 -> 17.8 mm, vias 8 -> 7
- net SDA: track 22.7 -> 19.1 mm
Other:
- board text added: "10/2014"
- board text added: "by PBAI & UWaterloo"
- board text added: "by PBAI and UWaterloo"
- board text removed: "08/2014"
