File: Hardware/PCB Design/Sound Board/Sound.brd (EAGLE design)
At the start: 68.2 x 80 mm, 63 parts

Commit message: Moved Sound Detector Board Pins
Spread out pins on sound detector boards so that the boards don’t
physically interfere with each other when 2 are mounted at the same
time.
Parts:
- moved SD_2 3.81 mm to (62.2, 36.8)
- moved C13 1.27 mm to (62.2, 74.9)
- moved SD_1 1.27 mm to (62.2, 62.9)
Routing:
- net DPEAK_2: track 60.3 -> 64.1 mm
- net 5VFILT: track 52.1 -> 55.4 mm
- net +5V_1: track 55.5 -> 53.2 mm
- net MIC_2: track 36.8 -> 35.6 mm
Changed lines of the file:
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@@
 <?xml version="1.0" encoding="utf-8"?>
 <!DOCTYPE eagle SYSTEM "eagle.dtd">
-<eagle version="7.1.0">
+<eagle version="7.0.0">
 <drawing>
 <settings>
@@
 <text x="41.91" y="40.005" size="1.778" layer="25">IN</text>
 <text x="34.925" y="40.005" size="1.778" layer="25">OUT</text>
-<text x="64.135" y="47.625" size="1.27" layer="26" rot="MR0">GND</text>
-<text x="64.135" y="68.58" size="1.27" layer="26" rot="MR0">GND</text>
+<text x="60.325" y="41.275" size="1.27" layer="26" rot="MR0">GND</text>
+<text x="60.325" y="67.31" size="1.27" layer="26" rot="MR0">GND</text>
 <text x="19.05" y="30.48" size="1.778" layer="25" rot="R90">Sound Module</text>
 <text x="21.59" y="30.48" size="1.27" layer="25" rot="R90">Hylozoic Series 3</text>
@@
 <attribute name="VALUE" x="65.405" y="66.675" size="0.762" layer="27" rot="R270"/>
 </element>
-<element name="C13" library="rcl" package="E5-10,5" value="470uF" x="62.23" y="73.66" smashed="yes" rot="R180">
-<attribute name="NAME" x="63.881" y="70.9168" size="1.27" layer="25" ratio="10" rot="R180"/>
-<attribute name="VALUE" x="65.3542" y="76.8858" size="1.27" layer="27" ratio="10" rot="R180"/>
+<element name="C13" library="rcl" package="E5-10,5" value="470uF" x="62.23" y="74.93" smashed="yes" rot="R180">
+<attribute name="NAME" x="63.881" y="72.1868" size="1.27" layer="25" ratio="10" rot="R180"/>
+<attribute name="VALUE" x="65.3542" y="78.1558" size="1.27" layer="27" ratio="10" rot="R180"/>
 </element>
 <element name="TAB_CONN" library="pinhead" package="2X05" value="" x="39.37" y="36.83" smashed="yes" rot="R180">
@@
 <attribute name="VALUE" x="45.72" y="41.275" size="1.27" layer="27" rot="R180"/>
 </element>
-<element name="SD_2" library="pinhead" package="1X05" value="" x="62.23" y="40.64" rot="MR90"/>
-<element name="SD_1" library="pinhead" package="1X05" value="" x="62.23" y="61.595" rot="MR90"/>
+<element name="SD_2" library="pinhead" package="1X05" value="" x="62.23" y="36.83" rot="MR90"/>
+<element name="SD_1" library="pinhead" package="1X05" value="" x="62.23" y="62.865" rot="MR90"/>
 <element name="JACK" library="CBLA_Test_bed_Library" package="RJ45-NO-SHIELD" value="RJ45-6L-B" x="25.4" y="73.66" smashed="yes" rot="R180">
 <attribute name="OC_NEWARK" value="16R6090" x="25.4" y="73.66" size="1.778" layer="27" rot="R180" display="off"/>
@@
 <wire x1="36.83" y1="60.96" x2="59.69" y2="60.96" width="0.4064" layer="16"/>
 <wire x1="59.69" y1="60.96" x2="59.69" y2="61.595" width="0.4064" layer="16"/>
-<wire x1="59.69" y1="61.595" x2="62.23" y2="61.595" width="0.4064" layer="16"/>
+<wire x1="59.69" y1="61.595" x2="62.23" y2="62.865" width="0.4064" layer="16"/>
 </signal>
 <signal name="FPWM_1_1">
@@
 <via x="36.83" y="48.26" extent="1-16" drill="0.7"/>
 <wire x1="36.83" y1="48.26" x2="59.69" y2="48.26" width="0.4064" layer="1"/>
-<wire x1="59.69" y1="48.26" x2="59.69" y2="40.64" width="0.4064" layer="1"/>
-<wire x1="59.69" y1="40.64" x2="62.23" y2="40.64" width="0.4064" layer="1"/>
+<wire x1="59.69" y1="48.26" x2="59.69" y2="36.83" width="0.4064" layer="1"/>
+<wire x1="59.69" y1="36.83" x2="62.23" y2="36.83" width="0.4064" layer="1"/>
 </signal>
 <signal name="DTRIG_1">
@@
 <contactref element="R15" pad="2"/>
 <wire x1="66.04" y1="62.65" x2="66.04" y2="31.75" width="0.8128" layer="1"/>
-<wire x1="66.04" y1="31.75" x2="63.5" y2="31.75" width="0.8128" layer="1"/>
-<via x="63.5" y="31.75" extent="1-16" drill="0.7"/>
-<wire x1="63.5" y1="31.75" x2="63.5" y2="19.05" width="0.8128" layer="16"/>
+<via x="66.04" y="31.75" extent="1-16" drill="0.7"/>
+<wire x1="66.04" y1="31.75" x2="63.5" y2="19.05" width="0.8128" layer="16"/>
 <via x="63.5" y="19.05" extent="1-16" drill="0.7"/>
 <wire x1="63.5" y1="19.05" x2="63.5" y2="17.36" width="0.8128" layer="1"/>
@@
 <wire x1="45.72" y1="58.42" x2="59.055" y2="58.42" width="0.4064" layer="16"/>
 <wire x1="59.055" y1="58.42" x2="59.055" y2="56.515" width="0.4064" layer="16"/>
-<wire x1="59.055" y1="56.515" x2="62.23" y2="56.515" width="0.4064" layer="16"/>
+<wire x1="59.055" y1="56.515" x2="62.23" y2="57.785" width="0.4064" layer="16"/>
 </signal>
 <signal name="MIC_2">
@@
 <wire x1="41.91" y1="38.1" x2="41.91" y2="42.545" width="0.4064" layer="1"/>
 <wire x1="41.91" y1="42.545" x2="57.15" y2="42.545" width="0.4064" layer="1"/>
-<wire x1="57.15" y1="42.545" x2="57.15" y2="33.02" width="0.4064" layer="1"/>
-<wire x1="57.15" y1="33.02" x2="62.23" y2="33.02" width="0.4064" layer="1"/>
-<wire x1="62.23" y1="33.02" x2="62.23" y2="35.56" width="0.4064" layer="1"/>
+<wire x1="57.15" y1="42.545" x2="57.15" y2="31.75" width="0.4064" layer="1"/>
+<wire x1="57.15" y1="31.75" x2="62.23" y2="31.75" width="0.4064" layer="1"/>
 </signal>
 <signal name="N$9">
@@
 <contactref element="SD_2" pad="4"/>
 <contactref element="TEENSY" pad="VIN"/>
-<wire x1="64.77" y1="73.66" x2="66.04" y2="73.66" width="0.4064" layer="1"/>
+<wire x1="64.77" y1="74.93" x2="66.04" y2="73.66" width="0.4064" layer="1"/>
 <wire x1="66.04" y1="73.66" x2="66.04" y2="64.35" width="0.4064" layer="1"/>
-<wire x1="64.77" y1="73.66" x2="64.77" y2="77.47" width="0.4064" layer="1"/>
+<wire x1="64.77" y1="74.93" x2="64.77" y2="77.47" width="0.4064" layer="1"/>
 <wire x1="64.77" y1="77.47" x2="54.61" y2="77.47" width="0.4064" layer="1"/>
-<wire x1="64.77" y1="43.18" x2="62.23" y2="43.18" width="0.4064" layer="1"/>
-<wire x1="62.23" y1="64.135" x2="64.77" y2="64.135" width="0.4064" layer="1"/>
-<wire x1="64.77" y1="64.135" x2="64.77" y2="63.5" width="0.4064" layer="1"/>
-<wire x1="64.77" y1="63.5" x2="64.77" y2="43.18" width="0.4064" layer="1"/>
+<wire x1="62.23" y1="65.405" x2="64.77" y2="64.135" width="0.4064" layer="1"/>
+<wire x1="64.77" y1="64.135" x2="64.77" y2="39.37" width="0.4064" layer="1"/>
 <wire x1="66.04" y1="64.35" x2="64.77" y2="64.35" width="0.4064" layer="1"/>
 <wire x1="64.77" y1="64.35" x2="64.77" y2="64.135" width="0.4064" layer="1"/>
+<wire x1="64.77" y1="39.37" x2="62.23" y2="39.37" width="0.4064" layer="1"/>
 </signal>
 <signal name="LED_JUMP_POW">
